File: kicad/pamp/compact.kicad_pcb (KiCad board)
At the start: 2 copper layers, 80 x 100 mm, 79 parts, among them J1 input, J2 Conn_01x02_Female, J3 output, J4 power, Q1 2SA1381F, Q10 BC546B, Q11 MJE340, Q12 2SA1381F, Q13 2SC3503F, Q14 BC546B, Q15 BC556B, Q16 IRFP240N, Q17 IRFP9240N, Q2 2SC3503F, Q3 2SA1381F, Q4 2SC3503F, Q5 BC550C, Q6 BC560C, Q7 BC550C, Q8 BC560C, Q9 BC556B

Commit message: Finished SPICE simulation, Kicad follows the updates
The VAS standing current was increased from 12mA to 15mA to avoid
VAS lower transistor switch-off during slewing. The VBE multiplier
was optimized for lower current-to-voltage dependency by increasing
collector resistor to 43 ohm. Also, the VBE resistor divider was
chosen in such way that we get around 8.9mV/C characteristic.

Kicad schematic was updated according to changes in Spice schematic.

Signed-off-by: Nenad Radulovic <nenad.b.radulovic@gmail.com>
Parts:
- removed D4, D5, D6: BAV21, Diode_THT:D_DO-41_SOD81_P7.62mm_Horizontal
- removed D7, D8: ZPY12-TR, Diode_THT:D_DO-41_SOD81_P10.16mm_Horizontal
- removed J4: power, TerminalBlock_Phoenix:TerminalBlock_Phoenix_MKDS-1,5-3-5.08_1x03_P5.08mm_Horizontal
- removed RV2: R_POT_TRIM, Potentiometer_THT:Potentiometer_ACP_CA9-V10_Vertical
- added C13: 100n, Capacitor_THT:C_Rect_L7.2mm_W5.5mm_P5.00mm_FKS2_FKP2_MKS2_MKP2, F.Cu at (186.6, 71.9)
- added C14: 100n, Capacitor_THT:C_Rect_L7.2mm_W5.5mm_P5.00mm_FKS2_FKP2_MKS2_MKP2, F.Cu at (194.3, 71.9)
- added C15: 470u, Capacitor_THT:CP_Radial_D10.0mm_P3.50mm, F.Cu at (178.2, 75.0)
- added C16: 470u, Capacitor_THT:CP_Radial_D10.0mm_P3.50mm, F.Cu at (196.1, 63.6)
- added Q18: MJL1302A, Package_TO_SOT_THT:TO-264-3_Vertical, F.Cu at (82.6, 32.5)
- added R32: 2R2, Resistor_THT:R_Axial_DIN0411_L9.9mm_D3.6mm_P12.70mm_Horizontal, F.Cu at (163.1, 71.3)
- added R33: 2R2, Resistor_THT:R_Axial_DIN0411_L9.9mm_D3.6mm_P12.70mm_Horizontal, F.Cu at (176.0, 45.2)
- added R34: 0.22, Resistor_THT:R_Box_L14.0mm_W5.0mm_P9.00mm, F.Cu at (164.8, 67.0)
- added R35: 0.22, Resistor_THT:R_Box_L14.0mm_W5.0mm_P9.00mm, F.Cu at (180.5, 62.8)
- added R36: 10, Resistor_THT:R_Axial_DIN0414_L11.9mm_D4.5mm_P5.08mm_Vertical, F.Cu at (163.5, 62.1)
- added R37: 4.7, Resistor_THT:R_Axial_DIN0411_L9.9mm_D3.6mm_P12.70mm_Horizontal, F.Cu at (184.1, 56.2)
- added R38: 10, Resistor_THT:R_Axial_DIN0207_L6.3mm_D2.5mm_P10.16mm_Horizontal, F.Cu at (163.1, 77.4)
- C1: value 100u -> 120p; footprint Capacitor_THT:CP_Radial_D10.0mm_P3.50mm -> Capacitor_THT:C_Disc_D8.0mm_W2.5mm_P5.00mm
- C10: value 100n -> 2u2; footprint Capacitor_THT:C_Rect_L7.2mm_W5.5mm_P5.00mm_FKS2_FKP2_MKS2_MKP2 -> Capacitor_THT:CP_Radial_D5.0mm_P2.50mm
- C11: value 470u -> 2u2; footprint Capacitor_THT:CP_Radial_D10.0mm_P3.50mm -> Capacitor_THT:CP_Radial_D5.0mm_P2.50mm
- C12: value 470u -> 100n; footprint Capacitor_THT:CP_Radial_D10.0mm_P3.50mm -> Capacitor_THT:C_Rect_L7.2mm_W5.5mm_P5.00mm_FKS2_FKP2_MKS2_MKP2
- C2: value 470p -> 100u; footprint Capacitor_THT:C_Disc_D3.8mm_W2.6mm_P2.50mm -> Capacitor_THT:CP_Radial_D10.0mm_P3.50mm
- C3: value 1m -> 120p; footprint Capacitor_THT:CP_Radial_D10.0mm_P3.50mm -> Capacitor_THT:C_Disc_D8.0mm_W2.5mm_P5.00mm
- C4: value 8.2p -> 1n2; footprint Capacitor_THT:C_Disc_D3.0mm_W2.0mm_P2.50mm -> Capacitor_THT:C_Disc_D8.0mm_W2.5mm_P5.00mm
- C5: value 47p -> 120p; footprint Capacitor_THT:C_Disc_D3.0mm_W2.0mm_P2.50mm -> Capacitor_THT:C_Disc_D8.0mm_W2.5mm_P5.00mm
- C6: value 47p -> 1m; footprint Capacitor_THT:C_Disc_D3.0mm_W2.0mm_P2.50mm -> Capacitor_THT:CP_Radial_D10.0mm_P3.50mm
- C7: value 47u -> 1n2; footprint Capacitor_THT:CP_Radial_D8.0mm_P2.50mm -> Capacitor_THT:C_Disc_D8.0mm_W2.5mm_P5.00mm
- C8: value 100n -> 8.2p; footprint Capacitor_THT:C_Rect_L7.2mm_W5.5mm_P5.00mm_FKS2_FKP2_MKS2_MKP2 -> Capacitor_THT:C_Disc_D3.0mm_W2.0mm_P2.50mm
- C9: value 100n -> 47u; footprint Capacitor_THT:C_Rect_L7.2mm_W5.5mm_P5.00mm_FKS2_FKP2_MKS2_MKP2 -> Capacitor_THT:CP_Radial_D6.3mm_P2.50mm
- J2: value Conn_01x02_Female -> power; footprint Connector_PinHeader_2.54mm:PinHeader_1x02_P2.54mm_Vertical -> TerminalBlock_Phoenix:TerminalBlock_Phoenix_MKDS-1,5-3-5.08_1x03_P5.08mm_Horizontal
- Q1: value 2SA1381F -> BC560C; footprint Package_TO_SOT_THT:TO-126-3_Vertical -> Package_TO_SOT_THT:TO-92L_Inline
- Q10, Q14: value BC546B -> BC556B
- Q11: value MJE340 -> 2SA1381F
- Q12: value 2SA1381F -> MJE340
- Q13: value 2SC3503F -> BC546B; footprint Package_TO_SOT_THT:TO-126-3_Vertical -> Package_TO_SOT_THT:TO-92L_Inline
- Q15: value BC556B -> 2SC4793; footprint Package_TO_SOT_THT:TO-92L_Inline -> Package_TO_SOT_THT:TO-220-3_Vertical
- Q16: value IRFP240N -> 2SA1837; footprint Package_TO_SOT_THT:TO-247-3_Vertical -> Package_TO_SOT_THT:TO-220-3_Vertical
- Q17: value IRFP9240N -> MJL3281A; footprint Package_TO_SOT_THT:TO-247-3_Vertical -> Package_TO_SOT_THT:TO-264-3_Vertical
- Q2, Q4: value 2SC3503F -> BC550C; footprint Package_TO_SOT_THT:TO-126-3_Vertical -> Package_TO_SOT_THT:TO-92L_Inline
- Q5: value BC550C -> BC560C
- Q6: value BC560C -> BC556B
- Q7: value BC550C -> BC546B
- Q8: value BC560C -> BC546B
- Q9: value BC556B -> 2SC3503F; footprint Package_TO_SOT_THT:TO-92L_Inline -> Package_TO_SOT_THT:TO-126-3_Vertical
- R1: value 10 -> 200
- R10, R22, R23: value 100 -> 1k5
- R12: value 100 -> 7k5; footprint Resistor_THT:R_Axial_DIN0207_L6.3mm_D2.5mm_P10.16mm_Horizontal -> Resistor_THT:R_Axial_DIN0411_L9.9mm_D3.6mm_P12.70mm_Horizontal
- R13, R25, R26: value 100 -> 22
- R15: value 1k5 -> 1k; footprint Resistor_THT:R_Axial_DIN0411_L9.9mm_D3.6mm_P12.70mm_Horizontal -> Resistor_THT:R_Axial_DIN0207_L6.3mm_D2.5mm_P10.16mm_Horizontal
- R16: value 6k8 -> 1k5; footprint Resistor_THT:R_Axial_DIN0207_L6.3mm_D2.5mm_P10.16mm_Horizontal -> Resistor_THT:R_Axial_DIN0411_L9.9mm_D3.6mm_P12.70mm_Horizontal
- R17: value 1k -> 43
- R18: value 18 -> 1k5
- R19: value 82 -> 270
- R2: value 10k -> 100
- R20: value 82 -> 43
- R21: value 18 -> 39k
- R24: value 100 -> 39k
- R27: value 100 -> 560
- R28: value 0.15 -> 560; footprint Resistor_THT:R_Box_L14.0mm_W5.0mm_P9.00mm -> Resistor_THT:R_Axial_DIN0207_L6.3mm_D2.5mm_P10.16mm_Horizontal
- R29: value 0.22 -> 1k2; footprint Resistor_THT:R_Box_L14.0mm_W5.0mm_P9.00mm -> Resistor_THT:R_Axial_DIN0207_L6.3mm_D2.5mm_P10.16mm_Horizontal
- R3: value 8k2 -> 100; footprint Resistor_THT:R_Axial_DIN0411_L9.9mm_D3.6mm_P12.70mm_Horizontal -> Resistor_THT:R_Axial_DIN0207_L6.3mm_D2.5mm_P10.16mm_Horizontal
- R30: value 10 -> 1k2; footprint Resistor_THT:R_Axial_DIN0411_L9.9mm_D3.6mm_P12.70mm_Horizontal -> Resistor_THT:R_Axial_DIN0207_L6.3mm_D2.5mm_P10.16mm_Horizontal
- R31: value 4.7 -> 51; footprint Resistor_THT:R_Axial_DIN0411_L9.9mm_D3.6mm_P12.70mm_Horizontal -> Resistor_THT:R_Axial_DIN0207_L6.3mm_D2.5mm_P10.16mm_Horizontal
- R4: value 100 -> 10k
- R5: value 1k -> 200
- R6: value 560 -> 100
- R7: value 1k5 -> 100
- R8: value 1k -> 7k5; footprint Resistor_THT:R_Axial_DIN0207_L6.3mm_D2.5mm_P10.16mm_Horizontal -> Resistor_THT:R_Axial_DIN0411_L9.9mm_D3.6mm_P12.70mm_Horizontal
- R9: value 100 -> 1k
- RV1: value R_POT_TRIM -> 1k
- moved C2 34.9 mm to (85.9, 87.2)
- moved Q15 14.6 mm to (113.2, 33.8), turned to 0 degrees
- moved Q16 11.9 mm to (101.7, 33.8)
- moved Q17 7.36 mm to (126.5, 32.5)
Connections:
- C1 pad 2: Net-(C1-Pad2) -> VSS
- C10 pad 1: GNDA -> Net-(C10-Pad1)
- C10 pad 2: VSS -> Net-(C10-Pad2)
- C11 pad 1: VDD -> Net-(C11-Pad1)
- C11 pad 2: GNDA -> Net-(C11-Pad2)
- C12 pad 1: GNDA -> Net-(C12-Pad1)
- C12 pad 2: VSS -> GNDA
- C2 pad 1: GNDS -> Net-(C2-Pad1)
- C3 pad 2: GNDS -> Net-(C3-Pad2)
- C4 pad 1: Net-(C4-Pad1) -> GNDS
- C4 pad 2: Net-(C4-Pad2) -> ninv
- C6 pad 2: Net-(C6-Pad2) -> GNDS
- C7 pad 1: Net-(C5-Pad2) -> Net-(C7-Pad1)
- C7 pad 2: Net-(C6-Pad1) -> Net-(C5-Pad1)
- C8 pad 1: Net-(C8-Pad1) -> preout
- C8 pad 2: GNDA -> inv
- C9 pad 1: VDD -> Net-(C9-Pad1)
- C9 pad 2: GNDA -> Net-(C7-Pad1)
- D1 pad 1: Net-(D1-Pad1) -> Net-(C7-Pad1)
- D1 pad 2: VDD -> Net-(C5-Pad2)
- D2 pad 2: Net-(D1-Pad1) -> Net-(C9-Pad1)
- D3 pad 1: Net-(D3-Pad1) -> Net-(C7-Pad1)
- J1 pad 3: Net-(C1-Pad2) -> Net-(C2-Pad2)
- J2 pad 1: Net-(J2-Pad1) -> VDD
- J2 pad 2: Net-(C6-Pad1) -> GNDA
- L1 pad 1: Net-(C4-Pad1) -> preout
- Q1 pad 1: Net-(D2-Pad1) -> Net-(C5-Pad2)
- Q1 pad 2: Net-(Q1-Pad2) -> ninv
- Q10 pad 1: Net-(C6-Pad2) -> Net-(Q10-Pad1)
- Q10 pad 3: VSS -> VDD
- Q11 pad 1: Net-(J2-Pad1) -> Net-(Q10-Pad2)
- Q11 pad 2: Net-(C5-Pad2) -> Net-(Q11-Pad2)
- Q11 pad 3: Net-(Q11-Pad3) -> Net-(Q10-Pad1)
- Q12 pad 1: Net-(Q12-Pad1) -> Net-(C7-Pad1)
- Q12 pad 2: Net-(C5-Pad2) -> Net-(C9-Pad1)
- Q12 pad 3: Net-(C5-Pad1) -> Net-(Q12-Pad3)
- Q13 pad 1: Net-(Q13-Pad1) -> Net-(D2-Pad1)
- Q13 pad 2: Net-(C6-Pad1) -> Net-(C10-Pad1)
- Q13 pad 3: Net-(C6-Pad2) -> preout
- Q14 pad 1: Net-(D5-Pad1) -> Net-(D3-Pad2)
- Q14 pad 2: Net-(Q14-Pad2) -> Net-(C11-Pad2)
- Q14 pad 3: Net-(C4-Pad1) -> preout
- Q15 pad 1: Net-(D6-Pad2) -> Net-(Q15-Pad1)
- Q15 pad 2: Net-(Q15-Pad2) -> VDD
- Q15 pad 3: Net-(C4-Pad1) -> Net-(Q15-Pad3)
- Q16 pad 2: VDD -> VSS
- Q16 pad 3: Net-(D7-Pad2) -> Net-(Q16-Pad3)
- Q17 pad 2: VSS -> VDD
- Q17 pad 3: Net-(D8-Pad1) -> Net-(Q17-Pad3)
- Q2 pad 1: Net-(D3-Pad2) -> Net-(C5-Pad2)
- Q2 pad 3: Net-(Q2-Pad3) -> Net-(C1-Pad1)
- Q3 pad 1: Net-(Q1-Pad3) -> Net-(Q3-Pad1)
- Q3 pad 3: Net-(Q1-Pad2) -> Net-(Q3-Pad3)
- Q4 pad 1: Net-(Q2-Pad3) -> Net-(Q2-Pad2)
- Q4 pad 2: Net-(Q4-Pad2) -> Net-(Q2-Pad2)
- Q4 pad 3: Net-(Q2-Pad2) -> Net-(C3-Pad2)
- Q5 pad 1: Net-(C5-Pad1) -> Net-(Q2-Pad2)
- Q5 pad 2: Net-(C2-Pad2) -> inv
- Q6 pad 1: Net-(C6-Pad2) -> Net-(Q3-Pad3)
- Q6 pad 2: Net-(C2-Pad2) -> Net-(Q3-Pad1)
- Q6 pad 3: Net-(Q6-Pad3) -> VDD
- Q7 pad 1: VDD -> Net-(C5-Pad2)
- Q7 pad 2: Net-(C4-Pad2) -> Net-(Q7-Pad2)
- Q7 pad 3: Net-(Q7-Pad3) -> VSS
- Q8 pad 1: VSS -> GNDA
- Q8 pad 2: Net-(C4-Pad2) -> Net-(C5-Pad2)
- Q9 pad 1: Net-(C5-Pad1) -> Net-(Q7-Pad2)
- Q9 pad 2: Net-(Q9-Pad2) -> Net-(C7-Pad1)
- Q9 pad 3: VDD -> Net-(Q8-Pad3)
- R1 pad 1: GNDA -> Net-(Q1-Pad3)
- R1 pad 2: GNDS -> Net-(Q3-Pad2)
- R10 pad 1: Net-(Q6-Pad3) -> ninv
- R10 pad 2: Net-(Q3-Pad2) -> GNDS
- R11 pad 2: Net-(C6-Pad2) -> Net-(Q8-Pad3)
- R12 pad 1: Net-(Q4-Pad2) -> GNDA
- R12 pad 2: Net-(Q7-Pad3) -> Net-(Q10-Pad1)
- R13 pad 1: Net-(Q8-Pad3) -> VSS
- R13 pad 2: Net-(Q3-Pad2) -> Net-(Q7-Pad2)
- R14 pad 1: Net-(C4-Pad2) -> inv
- R14 pad 2: Net-(C3-Pad1) -> Net-(C6-Pad1)
- R15 pad 1: Net-(C4-Pad2) -> Net-(C5-Pad1)
- R15 pad 2: Net-(C4-Pad1) -> preout
- R16 pad 1: Net-(Q11-Pad3) -> inv
- R16 pad 2: Net-(C5-Pad2) -> preout
- R17 pad 1: Net-(C6-Pad1) -> Net-(Q10-Pad2)
- R17 pad 2: Net-(R17-Pad2) -> VDD
- R18 pad 1: Net-(Q9-Pad2) -> Net-(Q12-Pad3)
- R18 pad 2: VDD -> Net-(Q11-Pad2)
- R19 pad 1: Net-(Q12-Pad1) -> Net-(C7-Pad1)
- R19 pad 2: Net-(Q9-Pad2) -> Net-(R19-Pad2)
- R2 pad 1: GNDS -> VSS
- R2 pad 2: Net-(C1-Pad2) -> Net-(C1-Pad1)
- R20 pad 1: Net-(Q10-Pad2) -> Net-(C9-Pad1)
- R20 pad 2: Net-(Q13-Pad1) -> Net-(Q11-Pad2)
- R21 pad 1: VSS -> Net-(C10-Pad1)
- R21 pad 2: Net-(Q10-Pad2) -> VDD
- R22 pad 1: Net-(Q16-Pad1) -> preout
- R22 pad 2: Net-(C5-Pad2) -> Net-(C10-Pad2)
- R23 pad 1: Net-(Q17-Pad1) -> Net-(C11-Pad1)
- R23 pad 2: Net-(C6-Pad1) -> preout
- R24 pad 1: Net-(C4-Pad1) -> VSS
- R24 pad 2: Net-(Q14-Pad2) -> Net-(C11-Pad2)
- R25 pad 1: Net-(Q15-Pad2) -> Net-(Q15-Pad1)
- R25 pad 2: Net-(C4-Pad1) -> Net-(C9-Pad1)
- R26 pad 1: Net-(D7-Pad2) -> Net-(Q16-Pad1)
- R26 pad 2: Net-(Q14-Pad2) -> Net-(C7-Pad1)
- R27 pad 1: Net-(D8-Pad1) -> preout
- R27 pad 2: Net-(Q15-Pad2) -> Net-(C10-Pad1)
- R28 pad 1: Net-(C4-Pad1) -> Net-(C11-Pad2)
- R28 pad 2: Net-(D7-Pad2) -> preout
- R29 pad 1: Net-(D8-Pad1) -> Net-(Q17-Pad3)
- R29 pad 2: Net-(C4-Pad1) -> Net-(C10-Pad1)
- R3 pad 1: Net-(Q2-Pad2) -> Net-(Q3-Pad1)
- R3 pad 2: Net-(Q1-Pad2) -> VDD
- R30 pad 1: Net-(C8-Pad1) -> Net-(Q18-Pad3)
- R30 pad 2: Net-(C4-Pad1) -> Net-(C11-Pad2)
- R31 pad 1: Net-(C4-Pad1) -> Net-(Q16-Pad3)
- R31 pad 2: Net-(J3-Pad1) -> Net-(Q15-Pad3)
- R4 pad 1: Net-(C2-Pad2) -> GNDS
- R4 pad 2: Net-(C1-Pad1) -> Net-(C2-Pad2)
- R5 pad 1: Net-(Q1-Pad3) -> Net-(Q5-Pad3)
- R5 pad 2: Net-(R5-Pad2) -> Net-(Q3-Pad2)
- R6 pad 2: Net-(Q2-Pad3) -> Net-(C3-Pad2)
- R7 pad 1: Net-(C2-Pad2) -> ninv
- R7 pad 2: GNDS -> Net-(C2-Pad1)
- R8 pad 1: Net-(C5-Pad1) -> GNDA
- R8 pad 2: VDD -> Net-(Q3-Pad3)
- R9 pad 1: Net-(Q4-Pad2) -> Net-(C3-Pad1)
- R9 pad 2: Net-(Q5-Pad3) -> GNDA
- RV1 pad 1: VDD -> Net-(Q12-Pad3)
- RV1 pad 2: VDD -> Net-(Q12-Pad3)
- RV1 pad 3: Net-(R5-Pad2) -> Net-(R19-Pad2)
