File: kicad/pamp/compact.sch (KiCad schematic (older format))
At the start: 2 parts

Commit message: WIP: Using symmetrical MOSFET design.
Signed-off-by: Nenad Radulovic <nenad.b.radulovic@gmail.com>
Parts:
- removed Q?: IRFP240, symbol Device:Q_NMOS_DGS
- added Q?: IRF9540N, Package_TO_SOT_THT:TO-220-3_Vertical, symbol Transistor_FET:IRF9540N
- added Q?: IRF540N, Package_TO_SOT_THT:TO-220-3_Vertical, symbol Transistor_FET:IRF540N
- added R? (x3): R, symbol Device:R
Other:
- moved on the sheet: R?
Changed lines of the file:
@@
 EESchema Schematic File Version 4
-EELAYER 26 0
+LIBS:compact-cache
+EELAYER 29 0
 EELAYER END
 $Descr A4 11693 8268
@@
 $EndDescr
 $Comp
-L Device:Q_NMOS_DGS Q?
-U 1 1 5C0A3FE8
-P 7300 2800
-F 0 "Q?" H 7505 2846 50  0000 L CNN
-F 1 "IRFP240" H 7505 2755 50  0000 L CNN
-F 2 "" H 7500 2900 50  0001 C CNN
-F 3 "~" H 7300 2800 50  0001 C CNN
-	1    7300 2800
+L Device:R R?
+U 1 1 5C0A407E
+P 6750 3000
+F 0 "R?" V 6543 3000 50  0000 C CNN
+F 1 "R" V 6634 3000 50  0000 C CNN
+F 2 "" V 6680 3000 50  0001 C CNN
+F 3 "~" H 6750 3000 50  0001 C CNN
+	1    6750 3000
+	0    1    1    0
+$EndComp
+$Comp
+L Device:R R?
+U 1 1 5CB45937
+P 7500 3750
+F 0 "R?" V 7293 3750 50  0000 C CNN
+F 1 "R" V 7384 3750 50  0000 C CNN
+F 2 "" V 7430 3750 50  0001 C CNN
+F 3 "~" H 7500 3750 50  0001 C CNN
+	1    7500 3750
+	-1   0    0    1
+$EndComp
+$Comp
+L Device:R R?
+U 1 1 5CB464D8
+P 7500 4250
+F 0 "R?" V 7293 4250 50  0000 C CNN
+F 1 "R" V 7384 4250 50  0000 C CNN
+F 2 "" V 7430 4250 50  0001 C CNN
+F 3 "~" H 7500 4250 50  0001 C CNN
+	1    7500 4250
+	-1   0    0    1
+$EndComp
+$Comp
+L Transistor_FET:IRF9540N Q?
+U 1 1 5CB4685B
+P 7400 5000
+F 0 "Q?" H 7606 4954 50  0000 L CNN
+F 1 "IRF9540N" H 7606 5045 50  0000 L CNN
+F 2 "Package_TO_SOT_THT:TO-220-3_Vertical" H 7600 4925 50  0001 L CIN
+F 3 "http://www.irf.com/product-info/datasheets/data/irf9540n.pdf" H 7400 5000 50  0001 L CNN
+	1    7400 5000
+	1    0    0    1
+$EndComp
+$Comp
+L Transistor_FET:IRF540N Q?
+U 1 1 5CB46DA9
+P 7400 3000
+F 0 "Q?" H 7606 3046 50  0000 L CNN
+F 1 "IRF540N" H 7606 2955 50  0000 L CNN
+F 2 "Package_TO_SOT_THT:TO-220-3_Vertical" H 7650 2925 50  0001 L CIN
+F 3 "http://www.irf.com/product-info/datasheets/data/irf540n.pdf" H 7400 3000 50  0001 L CNN
+	1    7400 3000
 	1    0    0    -1
 $EndComp
 $Comp
 L Device:R R?
-U 1 1 5C0A407E
-P 6850 2800
-F 0 "R?" V 6643 2800 50  0000 C CNN
-F 1 "R" V 6734 2800 50  0000 C CNN
-F 2 "" V 6780 2800 50  0001 C CNN
-F 3 "~" H 6850 2800 50  0001 C CNN
-	1    6850 2800
+U 1 1 5CB47763
+P 6750 5000
+F 0 "R?" V 6543 5000 50  0000 C CNN
+F 1 "R" V 6634 5000 50  0000 C CNN
+F 2 "" V 6680 5000 50  0001 C CNN
+F 3 "~" H 6750 5000 50  0001 C CNN
+	1    6750 5000
 	0    1    1    0
 $EndComp

Commit message: WIP: Started schematic.
Signed-off-by: Nenad Radulovic <nenad.b.radulovic@gmail.com>
Parts:
- removed R?: R, symbol Device:R
- added Q? (x2): MJE340, symbol Device:Q_NPN_BCE
- added R?: 100, symbol Device:R
- added R?: 6k8, symbol Device:R
- added R?: 560, symbol Device:R
- added RV?: R_POT_TRIM, symbol Device:R_POT_TRIM
- R?: value R -> 100; Power (none) -> 1/8; Type (none) -> MF
- R?: value R -> 0.15; Power (none) -> 5
- R?: value R -> 0.22; Power (none) -> 5
Connections:
- wire segments 0 -> 25
Changed lines of the file:
@@
 $Comp
 L Device:R R?
-U 1 1 5C0A407E
+U 0 0 5C0A407E
 P 6750 3000
-F 0 "R?" V 6543 3000 50  0000 C CNN
-F 1 "R" V 6634 3000 50  0000 C CNN
+F 0 "R?" V 6361 3000 50  0000 C CNN
+F 1 "100" V 6452 3000 50  0000 C CNN
 F 2 "" V 6680 3000 50  0001 C CNN
 F 3 "~" H 6750 3000 50  0001 C CNN
-	1    6750 3000
+F 4 "1/8" V 6543 3000 50  0000 C CNN "Power"
+F 5 "MF" V 6634 3000 50  0000 C CNN "Type"
+	0    6750 3000
 	0    1    1    0
 $EndComp
@@
 U 1 1 5CB45937
 P 7500 3750
-F 0 "R?" V 7293 3750 50  0000 C CNN
-F 1 "R" V 7384 3750 50  0000 C CNN
+F 0 "R?" H 7430 3659 50  0000 R CNN
+F 1 "0.15" H 7430 3750 50  0000 R CNN
 F 2 "" V 7430 3750 50  0001 C CNN
 F 3 "~" H 7500 3750 50  0001 C CNN
+F 4 "5" H 7430 3841 50  0000 R CNN "Power"
 	1    7500 3750
 	-1   0    0    1
@@
 U 1 1 5CB464D8
 P 7500 4250
-F 0 "R?" V 7293 4250 50  0000 C CNN
-F 1 "R" V 7384 4250 50  0000 C CNN
+F 0 "R?" H 7430 4159 50  0000 R CNN
+F 1 "0.22" H 7430 4250 50  0000 R CNN
 F 2 "" V 7430 4250 50  0001 C CNN
 F 3 "~" H 7500 4250 50  0001 C CNN
+F 4 "5" H 7430 4341 50  0000 R CNN "Power"
 	1    7500 4250
 	-1   0    0    1
@@
 	1    0    0    -1
 $EndComp
+Wire Wire Line
+	7500 3600 7500 3200
+Wire Wire Line
+	6900 3000 7200 3000
+Wire Wire Line
+	7500 4800 7500 4400
+Wire Wire Line
+	6900 5000 7200 5000
 $Comp
 L Device:R R?
-U 1 1 5CB47763
+U 0 0 5CB49D43
 P 6750 5000
-F 0 "R?" V 6543 5000 50  0000 C CNN
-F 1 "R" V 6634 5000 50  0000 C CNN
+F 0 "R?" V 6361 5000 50  0000 C CNN
+F 1 "100" V 6452 5000 50  0000 C CNN
 F 2 "" V 6680 5000 50  0001 C CNN
 F 3 "~" H 6750 5000 50  0001 C CNN
-	1    6750 5000
+F 4 "1/8" V 6543 5000 50  0000 C CNN "Power"
+F 5 "MF" V 6634 5000 50  0000 C CNN "Type"
+	0    6750 5000
 	0    1    1    0
 $EndComp
+$Comp
+L Device:Q_NPN_BCE Q?
+U 0 0 5CB4A062
+P 5900 3500
+F 0 "Q?" H 6091 3546 50  0000 L CNN
+F 1 "MJE340" H 6091 3455 50  0000 L CNN
+F 2 "" H 6100 3600 50  0001 C CNN
+F 3 "~" H 5900 3500 50  0001 C CNN
+	0    5900 3500
+	1    0    0    -1
+$EndComp
+$Comp
+L Device:Q_NPN_BCE Q?
+U 0 0 5CB4A3DF
+P 5900 4500
+F 0 "Q?" H 6091 4546 50  0000 L CNN
+F 1 "MJE340" H 6091 4455 50  0000 L CNN
+F 2 "" H 6100 4600 50  0001 C CNN
+F 3 "~" H 5900 4500 50  0001 C CNN
+	0    5900 4500
+	1    0    0    -1
+$EndComp
+$Comp
+L Device:R R?
+U 0 0 5CB4A5AF
+P 5000 3250
+F 0 "R?" H 4930 3113 50  0000 R CNN
+F 1 "6k8" H 4930 3204 50  0000 R CNN
+F 2 "" V 4930 3250 50  0001 C CNN
+F 3 "~" H 5000 3250 50  0001 C CNN
+F 4 "1/8" H 4930 3295 50  0000 R CNN "Power"
+F 5 "MF" H 4930 3386 50  0000 R CNN "Type"
+	0    5000 3250
+	-1   0    0    1
+$EndComp
+$Comp
+L Device:R R?
+U 0 0 5CB4B349
+P 5000 3750
+F 0 "R?" H 4930 3613 50  0000 R CNN
+F 1 "560" H 4930 3704 50  0000 R CNN
+F 2 "" V 4930 3750 50  0001 C CNN
+F 3 "~" H 5000 3750 50  0001 C CNN
+F 4 "1/8" H 4930 3795 50  0000 R CNN "Power"
+F 5 "MF" H 4930 3886 50  0000 R CNN "Type"
+	0    5000 3750
+	-1   0    0    1
+$EndComp
+$Comp
+L Device:R_POT_TRIM RV?
+U 1 1 5CB4C104
+P 5000 4750
+F 0 "RV?" H 4930 4796 50  0000 R CNN
+F 1 "R_POT_TRIM" H 4930 4705 50  0000 R CNN
+F 2 "" H 5000 4750 50  0001 C CNN
+F 3 "~" H 5000 4750 50  0001 C CNN
+	1    5000 4750
+	1    0    0    -1
+$EndComp
+Wire Wire Line
+	5700 4500 5500 4500
+Wire Wire Line
+	5500 4500 5500 4000
+Wire Wire Line
+	5500 4000 6000 4000
+Wire Wire Line
+	6000 4300 6000 4000
+Connection ~ 6000 4000
+Wire Wire Line
+	6000 4000 6000 3700
+Wire Wire Line
+	6000 4700 6000 5000
+Wire Wire Line
+	6000 5000 6600 5000
+Wire Wire Line
+	6000 5000 5000 5000
+Wire Wire Line
+	5000 5000 5000 4900
+Connection ~ 6000 5000
+Wire Wire Line
+	5000 4600 5000 4500
+Wire Wire Line
+	5150 4750 5250 4750
+Wire Wire Line
+	5250 4750 5250 4500
+Wire Wire Line
+	5250 4500 5000 4500
+Connection ~ 5000 4500
+Wire Wire Line
+	5000 4500 5000 3900
+Wire Wire Line
+	5000 3400 5000 3500
+Wire Wire Line
+	5700 3500 5000 3500
+Connection ~ 5000 3500
+Wire Wire Line
+	5000 3500 5000 3600
+Wire Wire Line
+	5000 3100 5000 3000
+Wire Wire Line
+	5000 3000 6000 3000
+Wire Wire Line
+	6000 3000 6000 3300
+Connection ~ 6000 3000
+Wire Wire Line
+	6000 3000 6600 3000
 $EndSCHEMATC

Commit message: WIP: Schematic is almost complete
Parts:
- added C?: 47u, symbol Device:CP
- added C? (x2): 47p, symbol Device:C
- added C?: 100n, symbol Device:C
- added C? (x2): 220u, symbol Device:CP
- added D? (x2): BAV21, symbol pspice:DIODE
- added D? (x4): 1N4148, symbol pspice:DIODE
- added D? (x2): BZX84C15, symbol Device:D_Zener
- added HS? (x2): Heatsink, symbol Mechanical:Heatsink
- added J? (x2): Screw_Terminal_01x03, symbol Connector:Screw_Terminal_01x03
- added J?: Screw_Terminal_01x02, symbol Connector:Screw_Terminal_01x02
- added Q?: BC546, symbol Device:Q_NPN_BCE
- added Q? (x7): Q_PNP_CBE, symbol Device:Q_PNP_CBE
- added Q? (x6): MJE340, symbol Device:Q_NPN_BCE
- added R? (x8): 100, symbol Device:R
- added R? (x2): 82, symbol Device:R
- added R? (x2): 20, symbol Device:R
- added R? (x2): 1k, symbol Device:R
- added R?: 560, symbol Device:R
- added R?: 470, symbol Device:R
- added R?: 8k2, symbol Device:R
- added R?: 10, symbol Device:R
- added RV?: 200, symbol Device:R_POT_TRIM
Connections:
- net labels added: GNDA, inn, inp, vdd, vss
- wire segments 25 -> 169
Other:
- moved on the sheet: Q?, R?, RV?

Commit message: Added all components.
Signed-off-by: Nenad Radulovic <nenad.b.radulovic@gmail.com>
Parts:
- added C10: 1000u, symbol Device:CP
- added C7, C8: 220p, symbol Device:C
- added C9: 100u, symbol Device:CP
- added L1: INDUCTOR, symbol pspice:INDUCTOR
- added R25: 10, symbol Device:R
- added R26, R29: 1k5, symbol Device:R
- added R27, R28: 100, symbol Device:R
- added R30, R31: 10k, symbol Device:R
- gave numbers to parts that had none: 63
Connections:
- net labels added: GNDS, input, out, preout
- wire segments 169 -> 219
Other:
- moved on the sheet: J1, J2, J3

Commit message: WIP: Resolving ERC.
Signed-off-by: Nenad Radulovic <nenad.b.radulovic@gmail.com>
Parts:
- removed Q11, Q3: Q_PNP_CBE, symbol Device:Q_PNP_CBE
- removed Q14, Q4: MJE340, symbol Device:Q_NPN_BCE
- removed Q15: BC546, symbol Device:Q_NPN_BCE
- added Q11, Q3: 2SA1381F, Package_TO_SOT_THT:TO-126-3_Vertical, symbol Device:Q_PNP_ECB
- added Q14, Q4: 2SC3503F, Package_TO_SOT_THT:TO-126-3_Vertical, symbol Device:Q_NPN_ECB
- added Q15: BC546B, Package_TO_SOT_THT:TO-92L_Inline, symbol Device:Q_NPN_CBE
- C1, C2: footprint (none) -> Capacitor_THT:C_Disc_D3.0mm_W2.0mm_P2.50mm
- C10: footprint (none) -> Capacitor_THT:CP_Radial_D8.0mm_P3.50mm
- C3: footprint (none) -> Capacitor_THT:CP_Radial_D6.3mm_P2.50mm
- C4, C5: footprint (none) -> Capacitor_THT:CP_Radial_D10.0mm_P3.80mm
- C6: footprint (none) -> Capacitor_THT:C_Rect_L7.2mm_W3.5mm_P5.00mm_FKS2_FKP2_MKS2_MKP2
- C7, C8: footprint (none) -> Capacitor_THT:C_Disc_D3.4mm_W2.1mm_P2.50mm
- C9: footprint (none) -> Capacitor_THT:CP_Radial_D8.0mm_P2.50mm
- D1, D2, D3, D4, D5, D6: footprint (none) -> Diode_THT:D_DO-41_SOD81_P7.62mm_Horizontal
- D7, D8: footprint (none) -> Diode_THT:D_DO-41_SOD81_P10.16mm_Horizontal
- HS1, HS2: footprint (none) -> Heatsink:Heatsink_Stonecold_HS-132_32x14mm_2xFixation1.5mm; symbol Mechanical:Heatsink -> Mechanical:Heatsink_Pad
- J1, J3: footprint (none) -> TerminalBlock_Phoenix:TerminalBlock_Phoenix_MKDS-1,5-3_1x03_P5.00mm_Horizontal
- J2: footprint (none) -> TerminalBlock_Phoenix:TerminalBlock_Phoenix_MKDS-1,5-2_1x02_P5.00mm_Horizontal
- L1: footprint (none) -> Inductor_THT:L_Axial_L26.7mm_D14.0mm_P7.62mm_Vertical_Vishay_IHA-104
- Q1: value Q_PNP_CBE -> 2SA1381F; footprint (none) -> Package_TO_SOT_THT:TO-126-3_Vertical; symbol Device:Q_PNP_CBE -> Device:Q_PNP_ECB
- Q10: value MJE340 -> BC546B; footprint (none) -> Package_TO_SOT_THT:TO-92L_Inline; symbol Device:Q_NPN_BCE -> Device:Q_NPN_CBE
- Q12, Q13: footprint (none) -> Package_TO_SOT_THT:TO-126-3_Vertical
- Q16, Q9: value Q_PNP_CBE -> BC556B; footprint (none) -> Package_TO_SOT_THT:TO-92L_Inline
- Q17: value IRF540N -> IRFP240N; footprint Package_TO_SOT_THT:TO-220-3_Vertical -> Package_TO_SOT_THT:TO-247-3_Vertical
- Q18: value IRF9540N -> IRFP9240N; footprint Package_TO_SOT_THT:TO-220-3_Vertical -> Package_TO_SOT_THT:TO-247-3_Vertical
- Q2: value MJE340 -> 2SC3503F; footprint (none) -> Package_TO_SOT_THT:TO-126-3_Vertical; symbol Device:Q_NPN_BCE -> Device:Q_NPN_ECB
- Q5, Q7: value MJE340 -> BC550C; footprint (none) -> Package_TO_SOT_THT:TO-92L_Inline; symbol Device:Q_NPN_BCE -> Device:Q_NPN_CBE
- Q6, Q8: value Q_PNP_CBE -> BC560C; footprint (none) -> Package_TO_SOT_THT:TO-92L_Inline
- R1, R10, R11, R12, R13, R14, R15, R16, R17, R18, R19, R2, R20, R21, R22, R23, R24, R25, R26, R27, R28, R29, R3, R30, R31, R4, R5, R6, R7, R8, R9: footprint (none) -> Resistor_THT:R_Axial_DIN0207_L6.3mm_D2.5mm_P10.16mm_Horizontal
- RV1: footprint (none) -> Potentiometer_THT:Potentiometer_ACP_CA9-V10_Vertical
- RV2: value R_POT_TRIM -> 1k; footprint (none) -> Potentiometer_THT:Potentiometer_ACP_CA9-V10_Vertical
Connections:
- wire segments 219 -> 220
Other:
- moved on the sheet: R1
